File: pcb/pcb.sch (KiCad schematic (older format))
At the start: 0 parts

Commit message: finish sch rev 0.1
Other:
- note added: "EINK"
- note removed: "STN LCD"
Changed lines of the file:
@@
 EESchema Schematic File Version 4
-LIBS:pcb-cache
 EELAYER 30 0
 EELAYER END
@@
 MCU
 Text Notes 1700 3350 0    100  ~ 0
-STN LCD
+EINK
 Text Notes 1700 2550 0    100  ~ 0
 TF-Card
