File: pcb/power.sch (KiCad schematic (older format))
At the start: 48 parts, among them SW1 SW_SP3T, U1 LTC3553, U100 LPC5500, Y1 32.768kHz, Y2 24MHz

Commit message: finish sch rev 0.1
Parts:
- removed BT1: Battery, footprints:BatteryHolder_Keystone_5204_5226, symbol Device:Battery
- removed C23, C25, C26, C27, C28, C29: 100nF, Capacitor_SMD:C_0402_1005Metric, symbol Device:C
- removed C42: 100uF, Capacitor_SMD:C_Elec_5x5.4, symbol Device:CP
- removed L2: 4.7uH, Inductor_SMD:L_Vishay_IHLP-1212, symbol Device:L
- removed U1: LTC3553, Package_DFN_QFN:QFN-20-1EP_3x3mm_P0.4mm_EP1.65x1.65mm, symbol Battery_Management:LTC3553
- removed U100: LPC5500, Package_QFP:TQFP-100-1EP_14x14mm_P0.5mm_EP5x5mm_ThermalVias, symbol symbols:LPC5500
- added BT1: JST2.0, symbol Device:Battery_Cell
- added C8: 220pF, Capacitor_SMD:C_0402_1005Metric, symbol Device:C
- added C9: 2.2uF, Capacitor_SMD:C_0603_1608Metric, symbol Device:C
- added R8: 1.87K, Resistor_SMD:R_0603_1608Metric, symbol Device:R
- added R9: 100K, Resistor_SMD:R_0603_1608Metric, symbol Device:R
- added TH1: 100K, symbol Device:Thermistor_NTC
- added U1: LTC3554, Package_DFN_QFN:VQFN-20-1EP_3x3mm_P0.4mm_EP1.7x1.7mm_ThermalVias, symbol symbols:LTC3554
- added U100: LPC5500_FBD64, Package_QFP:LQFP-64-1EP_10x10mm_P0.5mm_EP5x5mm_ThermalVias, symbol symbols:LPC5500_FBD64
- added U2: LTC2942-1, Package_DFN_QFN:DFN-6-1EP_3x2mm_P0.5mm_EP1.65x1.35mm, symbol Battery_Management:LTC2942-1
- C1: value 4.7uF -> 10uF
- C5: value 22uF -> 10uF
- L3: value 10uH -> 4.7uH
- R2: value 100K -> 2.05M
- R3: value 80.6K -> 649K
- R5: value 100K -> 1M
- renumbered C8 to C10
Connections:
- net labels added: +2V0, +SYS, CHRG, I2C1_SCL, I2C1_SDA, STBY
- net labels removed: +1V8, BAT_LOW, EXT_PWR_GOOD
- wire segments 145 -> 142
Other:
- note added: "PGOOD is OD output, no need to extra diode"
- note removed: "Maximum 150mA\n(Voltage drop 7.5mV)"
- moved on the sheet: C1, C2, C20, C21, C22, C3, C4, C5, C6, C7, L1, L3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

Commit message: assign footprints
Parts:
- BT1: footprint (none) -> Connector_JST:JST_PH_B2B-PH-K_1x02_P2.00mm_Vertical
- C9: footprint Capacitor_SMD:C_0603_1608Metric -> Capacitor_SMD:C_0402_1005Metric
- TH1: footprint (none) -> Resistor_SMD:R_0603_1608Metric
- Y1: value 32.768kHz -> DNP/32.768kHz
Changed lines of the file:
@@
 P 7850 2000
 F 0 "Y1" H 7850 2250 50  0000 C CNN
-F 1 "32.768kHz" H 7850 2150 50  0000 C CNN
+F 1 "DNP/32.768kHz" H 7850 2150 50  0000 C CNN
 F 2 "Crystal:Crystal_SMD_TXC_9HT11-2Pin_2.0x1.2mm_HandSoldering" H 7850 2000 50  0001 C CNN
 F 3 "~" H 7850 2000 50  0001 C CNN
@@
 F 0 "BT1" H 3168 5046 50  0000 L CNN
 F 1 "JST2.0" H 3168 4955 50  0000 L CNN
-F 2 "" V 3050 5010 50  0001 C CNN
+F 2 "Connector_JST:JST_PH_B2B-PH-K_1x02_P2.00mm_Vertical" V 3050 5010 50  0001 C CNN
 F 3 "~" V 3050 5010 50  0001 C CNN
 	1    3050 4950
@@
 F 0 "TH1" H 3598 5246 50  0000 L CNN
 F 1 "100K" H 3598 5155 50  0000 L CNN
-F 2 "" H 3500 5250 50  0001 C CNN
+F 2 "Resistor_SMD:R_0603_1608Metric" H 3500 5250 50  0001 C CNN
 F 3 "~" H 3500 5250 50  0001 C CNN
 	1    3500 5200
@@
 F 0 "C9" V 6900 4650 50  0000 L CNN
 F 1 "2.2uF" V 6900 4950 50  0000 L CNN
-F 2 "Capacitor_SMD:C_0603_1608Metric" H 6988 4700 50  0001 C CNN
+F 2 "Capacitor_SMD:C_0402_1005Metric" H 6988 4700 50  0001 C CNN
 F 3 "~" H 6950 4850 50  0001 C CNN
 	1    6950 4850

Commit message: rev 0.1
Parts:
- removed SW1: SW_SP3T, footprints:SW_SP3T_JSM0701SAQNL, symbol Switch:SW_SP3T
- added C13: 10uF, Capacitor_SMD:C_0603_1608Metric, symbol Device:C
- added SW1: SW_Push, Button_Switch_SMD:SW_SPST_EVQP7C, symbol Switch:SW_Push
- BT1: value JST2.0 -> Molex1.25; footprint Connector_JST:JST_PH_B2B-PH-K_1x02_P2.00mm_Vertical -> Connector_Molex:Molex_PicoBlade_53261-0271_1x02-1MP_P1.25mm_Horizontal
Connections:
- net GND: now also C13.2, SW1.1
- net PWR_KEY: now also SW1.2
- net at U1.17 (VBAT), U2.1 (SENSE+): now also C13.1
- no-connect marks 1 -> 0
Changed lines of the file:
@@
 L power:GND #PWR0318
 U 1 1 5D830E91
-P 4000 5250
-F 0 "#PWR0318" H 4000 5000 50  0001 C CNN
-F 1 "GND" H 4005 5077 50  0000 C CNN
-F 2 "" H 4000 5250 50  0001 C CNN
-F 3 "" H 4000 5250 50  0001 C CNN
-	1    4000 5250
+P 4100 5150
+F 0 "#PWR0318" H 4100 4900 50  0001 C CNN
+F 1 "GND" H 4105 4977 50  0000 C CNN
+F 2 "" H 4100 5150 50  0001 C CNN
+F 3 "" H 4100 5150 50  0001 C CNN
+	1    4100 5150
 	-1   0    0    -1
 $EndComp
@@
 PWR_KEY
 Wire Wire Line
-	5200 5050 4500 5050
-Wire Wire Line
-	4100 5150 4000 5150
-Wire Wire Line
-	4000 5150 4000 5250
-NoConn ~ 4100 5050
-$Comp
-L Switch:SW_SP3T SW1
-U 1 1 5D24F9B8
-P 4300 5050
-F 0 "SW1" H 4300 5333 50  0000 C CNN
-F 1 "SW_SP3T" H 4300 5242 50  0000 C CNN
-F 2 "footprints:SW_SP3T_JSM0701SAQNL" H 3675 5225 50  0001 C CNN
-F 3 "~" H 3675 5225 50  0001 C CNN
-	1    4300 5050
-	-1   0    0    -1
-$EndComp
-Text GLabel 4100 4950 0    50   Output ~ 0
-HOLD
+	4200 5050 4100 5050
+Wire Wire Line
+	4100 5050 4100 5150
 Wire Wire Line
 	6600 5650 6700 5650
@@
 Wire Wire Line
 	6900 2100 6600 2100
-$Comp
-L Device:L L5
-U 1 1 5D92C52E
-P 2850 1300
-F 0 "L5" V 3040 1300 50  0000 C CNN
-F 1 "MI0603J601R-10" V 2949 1300 50  0000 C CNN
-F 2 "Inductor_SMD:L_0603_1608Metric" H 2850 1300 50  0001 C CNN
-F 3 "~" H 2850 1300 50  0001 C CNN
-	1    2850 1300
-	0    -1   -1   0
-$EndComp
 Wire Wire Line
 	5100 1300 5200 1300
@@
 Wire Wire Line
 	2600 1200 2600 1300
-Wire Wire Line
-	2600 1300 2700 1300
 Connection ~ 2600 1300
 Wire Wire Line
@@
 	5200 2800 5100 2800
 Wire Wire Line
-	5200 3000 5100 3000
-Wire Wire Line
-	5100 3000 5100 2900
-Wire Wire Line
 	5200 2900 5100 2900
-Connection ~ 5100 2900
 Wire Wire Line
 	5100 2900 5100 2800
@@
 P 3050 4950
 F 0 "BT1" H 3168 5046 50  0000 L CNN
-F 1 "JST2.0" H 3168 4955 50  0000 L CNN
-F 2 "Connector_JST:JST_PH_B2B-PH-K_1x02_P2.00mm_Vertical" V 3050 5010 50  0001 C CNN
+F 1 "Molex1.25" H 3168 4955 50  0000 L CNN
+F 2 "Connector_Molex:Molex_PicoBlade_53261-0271_1x02-1MP_P1.25mm_Horizontal" V 3050 5010 50  0001 C CNN
 F 3 "~" V 3050 5010 50  0001 C CNN
 	1    3050 4950
@@
 U 1 1 5E78AA4A
 P 5900 4850
+AR Path="/5E78AA4A" Ref="U1"  Part="1"
+AR Path="/5D4C99F9/5E78AA4A" Ref="U1"  Part="1"
 F 0 "U1" H 5900 5915 50  0000 C CNN
 F 1 "LTC3554" H 5900 5824 50  0000 C CNN
@@
 	1    0    0    -1
 $EndComp
-$Comp
-L power:GND #PWR0134
-U 1 1 5E8951C8
-P 4400 5050
-F 0 "#PWR0134" H 4400 4800 50  0001 C CNN
-F 1 "GND" H 4405 4877 50  0000 C CNN
-F 2 "" H 4400 5050 50  0001 C CNN
-F 3 "" H 4400 5050 50  0001 C CNN
-	1    4400 5050
-	1    0    0    -1
-$EndComp
 Wire Wire Line
 	5200 5450 5100 5450
@@
 	0    1    1    0
 $EndComp
-$Comp
-L symbols:LPC5500_FBD64 U100
-U 2 1 5E9C51BB
-P 5900 1400
-F 0 "U100" H 5900 1765 50  0000 C CNN
-F 1 "LPC5500_FBD64" H 5900 1674 50  0000 C CNN
-F 2 "Package_QFP:LQFP-64-1EP_10x10mm_P0.5mm_EP5x5mm_ThermalVias" H 5900 1800 50  0001 C CNN
-F 3 "" H 5800 1450 50  0001 C CNN
-	2    5900 1400
-	1    0    0    -1
-$EndComp
 Wire Wire Line
 	6700 2800 6700 3000
@@
 Wire Wire Line
 	4300 1300 4700 1300
-Wire Wire Line
-	3000 1300 3500 1300
 Text Notes 7100 4650 0    50   ~ 0
 PGOOD is OD output, no need to extra diode
@@
 Wire Wire Line
 	2500 4400 2900 4400
+$Comp
+L Switch:SW_Push SW?
+U 1 1 5E820CD6
+P 4400 5050
+AR Path="/5D438406/5E820CD6" Ref="SW?"  Part="1"
+AR Path="/5D4C99F9/5E820CD6" Ref="SW1"  Part="1"
+F 0 "SW1" H 4400 5335 50  0000 C CNN
+F 1 "SW_Push" H 4400 5244 50  0000 C CNN
+F 2 "Button_Switch_SMD:SW_SPST_EVQP7C" H 4400 5250 50  0001 C CNN
+F 3 "~" H 4400 5250 50  0001 C CNN
+	1    4400 5050
+	1    0    0    -1
+$EndComp
+Wire Wire Line
+	3000 1300 3500 1300
+Wire Wire Line
+	2600 1300 2700 1300
+$Comp
+L Device:L L5
+U 1 1 5D92C52E
+P 2850 1300
+F 0 "L5" V 3040 1300 50  0000 C CNN
+F 1 "MI0603J601R-10" V 2949 1300 50  0000 C CNN
+F 2 "Inductor_SMD:L_0603_1608Metric" H 2850 1300 50  0001 C CNN
+F 3 "~" H 2850 1300 50  0001 C CNN
+	1    2850 1300
+	0    -1   -1   0
+$EndComp
+$Comp
+L symbols:LPC5500_FBD64 U100
+U 2 1 5E9C51BB
+P 5900 1400
+AR Path="/5E9C51BB" Ref="U100"  Part="2"
+AR Path="/5D4C99F9/5E9C51BB" Ref="U100"  Part="2"
+F 0 "U100" H 5900 1765 50  0000 C CNN
+F 1 "LPC5500_FBD64" H 5900 1674 50  0000 C CNN
+F 2 "Package_QFP:LQFP-64-1EP_10x10mm_P0.5mm_EP5x5mm_ThermalVias" H 5900 1800 50  0001 C CNN
+F 3 "" H 5800 1450 50  0001 C CNN
+	2    5900 1400
+	1    0    0    -1
+$EndComp
+$Comp
+L Device:C C13
+U 1 1 5EBEB32F
+P 4000 4900
+F 0 "C13" H 3800 4900 50  0000 L CNN
+F 1 "10uF" H 3750 4800 50  0000 L CNN
+F 2 "Capacitor_SMD:C_0603_1608Metric" H 4038 4750 50  0001 C CNN
+F 3 "~" H 4000 4900 50  0001 C CNN
+	1    4000 4900
+	1    0    0    -1
+$EndComp
+$Comp
+L power:GND #PWR0117
+U 1 1 5EBEB335
+P 4000 5050
+F 0 "#PWR0117" H 4000 4800 50  0001 C CNN
+F 1 "GND" H 4005 4877 50  0000 C CNN
+F 2 "" H 4000 5050 50  0001 C CNN
+F 3 "" H 4000 5050 50  0001 C CNN
+	1    4000 5050
+	1    0    0    -1
+$EndComp
+Wire Wire Line
+	4600 5050 5200 5050
+Connection ~ 4000 4750
 $EndSCHEMATC

Commit message: pcb: bug fixes
Parts:
- removed BT1: Molex1.25, Connector_Molex:Molex_PicoBlade_53261-0271_1x02-1MP_P1.25mm_Horizontal, symbol Device:Battery_Cell
- added BT1: Conn_01x02, Connector_Molex:Molex_PicoBlade_53261-0271_1x02-1MP_P1.25mm_Horizontal, symbol Connector_Generic:Conn_01x02
- L1: value 10uH -> 6.8uH
- R6: value 80.6K -> 649K
- Y2: value 24MHz -> 16MHz
Connections:
- net STBY is gone; now on net GND: U1.10 (STBY)
- net +BATT: now also BT1.2 (Pin_2)
- net GND: now also BT1.1 (Pin_1)
Changed lines of the file:
@@
 P 7150 5700
 F 0 "L1" V 7200 5550 50  0000 C CNN
-F 1 "10uH" V 7200 5850 50  0000 C CNN
+F 1 "6.8uH" V 7200 5850 50  0000 C CNN
 F 2 "Inductor_SMD:L_Vishay_IHLP-1212" H 7150 5700 50  0001 C CNN
 F 3 "~" H 7150 5700 50  0001 C CNN
@@
 P 7400 6150
 F 0 "R6" H 7200 6200 50  0000 L CNN
-F 1 "80.6K" H 7100 6100 50  0000 L CNN
+F 1 "649K" H 7100 6100 50  0000 L CNN
 F 2 "Resistor_SMD:R_0603_1608Metric" V 7330 6150 50  0001 C CNN
 F 3 "~" H 7400 6150 50  0001 C CNN
@@
 Text GLabel 6800 4550 2    50   Output ~ 0
 PB_STAT
-Text GLabel 5000 5350 0    50   Input ~ 0
+Text GLabel 4900 5350 0    50   Input ~ 0
 PMIC_ON_REQ
 Text GLabel 6800 4650 2    50   Output ~ 0
@@
 Wire Wire Line
 	6600 4650 6800 4650
-Wire Wire Line
-	5200 5350 5100 5350
 $Comp
 L Device:C C5
@@
 P 8650 1700
 F 0 "Y2" H 8550 2000 50  0000 L CNN
-F 1 "24MHz" H 8500 1900 50  0000 L CNN
+F 1 "16MHz" H 8500 1900 50  0000 L CNN
 F 2 "Oscillator:Oscillator_SMD_Abracon_ASE-4Pin_3.2x2.5mm" H 8650 1700 50  0001 C CNN
 F 3 "~" H 8650 1700 50  0001 C CNN
@@
 $EndComp
 $Comp
-L Device:Battery_Cell BT1
-U 1 1 5E789CDC
-P 3050 4950
-F 0 "BT1" H 3168 5046 50  0000 L CNN
-F 1 "Molex1.25" H 3168 4955 50  0000 L CNN
-F 2 "Connector_Molex:Molex_PicoBlade_53261-0271_1x02-1MP_P1.25mm_Horizontal" V 3050 5010 50  0001 C CNN
-F 3 "~" V 3050 5010 50  0001 C CNN
-	1    3050 4950
-	1    0    0    -1
-$EndComp
-$Comp
 L symbols:LTC3554 U1
 U 1 1 5E78AA4A
@@
 $EndComp
 Wire Wire Line
-	5200 5450 5100 5450
-Wire Wire Line
-	5100 5450 5100 5350
-Connection ~ 5100 5350
-Wire Wire Line
-	5100 5350 5000 5350
-Text GLabel 5000 5150 0    50   Input ~ 0
-STBY
-Wire Wire Line
-	5000 5150 5200 5150
+	5000 5450 5000 5350
+Connection ~ 5000 5350
+Wire Wire Line
+	5000 5350 4900 5350
 Connection ~ 3050 4750
 $Comp
 L power:GND #PWR0145
 U 1 1 5E8C89CD
-P 3050 5050
-F 0 "#PWR0145" H 3050 4800 50  0001 C CNN
-F 1 "GND" H 3055 4877 50  0000 C CNN
-F 2 "" H 3050 5050 50  0001 C CNN
-F 3 "" H 3050 5050 50  0001 C CNN
-	1    3050 5050
+P 3050 4850
+F 0 "#PWR0145" H 3050 4600 50  0001 C CNN
+F 1 "GND" H 3055 4677 50  0000 C CNN
+F 2 "" H 3050 4850 50  0001 C CNN
+F 3 "" H 3050 4850 50  0001 C CNN
+	1    3050 4850
 	1    0    0    -1
 $EndComp
@@
 	4600 5050 5200 5050
 Connection ~ 4000 4750
+Wire Wire Line
+	5000 5350 5200 5350
+Wire Wire Line
+	5000 5450 5200 5450
+Wire Wire Line
+	5200 5150 5100 5150
+Wire Wire Line
+	5100 5150 5100 5650
+Connection ~ 5100 5650
+$Comp
+L Connector_Generic:Conn_01x02 BT1
+U 1 1 5E820C63
+P 2850 4850
+F 0 "BT1" H 3200 4750 50  0000 C CNN
+F 1 "Conn_01x02" H 3200 4850 50  0000 C CNN
+F 2 "Connector_Molex:Molex_PicoBlade_53261-0271_1x02-1MP_P1.25mm_Horizontal" H 2850 4850 50  0001 C CNN
+F 3 "~" H 2850 4850 50  0001 C CNN
+	1    2850 4850
+	-1   0    0    1
+$EndComp
 $EndSCHEMATC

Commit message: pcb: rev 0.2
Parts:
- removed Y1: DNP/32.768kHz, Crystal:Crystal_SMD_TXC_9HT11-2Pin_2.0x1.2mm_HandSoldering, symbol Device:Crystal
- C2, C7: value 100uF -> 47uF; footprint Capacitor_SMD:C_1206_3216Metric -> Capacitor_SMD:C_0805_2012Metric
- C3: value 10uF -> 1uF; footprint Capacitor_SMD:C_0603_1608Metric -> Capacitor_SMD:C_0402_1005Metric
- L1: value 6.8uH -> 10uH
- R4, R7: value 0R05 -> 0/0R05; footprint Resistor_SMD:R_1206_3216Metric -> Resistor_SMD:R_0805_2012Metric
Connections:
- no-connect marks 0 -> 2
Changed lines of the file:
@@
 Sheet 3 8
 Title "Bric"
-Date "2020-03-09"
-Rev "R0.1"
+Date "2020-03-25"
+Rev "R0.2"
 Comp "EE300"
 Comment1 "zephray@outlook.com"
@@
 P 7150 5700
 F 0 "L1" V 7200 5550 50  0000 C CNN
-F 1 "6.8uH" V 7200 5850 50  0000 C CNN
+F 1 "10uH" V 7200 5850 50  0000 C CNN
 F 2 "Inductor_SMD:L_Vishay_IHLP-1212" H 7150 5700 50  0001 C CNN
 F 3 "~" H 7150 5700 50  0001 C CNN
@@
 P 8200 5850
 F 0 "C3" H 7950 5900 50  0000 L CNN
-F 1 "10uF" H 7900 5800 50  0000 L CNN
-F 2 "Capacitor_SMD:C_0603_1608Metric" H 8238 5700 50  0001 C CNN
+F 1 "1uF" H 7900 5800 50  0000 L CNN
+F 2 "Capacitor_SMD:C_0402_1005Metric" H 8238 5700 50  0001 C CNN
 F 3 "~" H 8200 5850 50  0001 C CNN
 	1    8200 5850
@@
 P 8450 5700
 F 0 "R4" V 8250 5700 50  0000 C CNN
-F 1 "0R05" V 8350 5700 50  0000 C CNN
-F 2 "Resistor_SMD:R_1206_3216Metric" V 8380 5700 50  0001 C CNN
+F 1 "0/0R05" V 8350 5700 50  0000 C CNN
+F 2 "Resistor_SMD:R_0805_2012Metric" V 8380 5700 50  0001 C CNN
 F 3 "~" H 8450 5700 50  0001 C CNN
 	1    8450 5700
@@
 P 8700 5850
 F 0 "C2" H 8450 5900 50  0000 L CNN
-F 1 "100uF" H 8300 5800 50  0000 L CNN
-F 2 "Capacitor_SMD:C_1206_3216Metric" H 8738 5700 50  0001 C CNN
+F 1 "47uF" H 8300 5800 50  0000 L CNN
+F 2 "Capacitor_SMD:C_0805_2012Metric" H 8738 5700 50  0001 C CNN
 F 3 "~" H 8700 5850 50  0001 C CNN
 	1    8700 5850
@@
 P 8450 4950
 F 0 "R7" V 8250 4950 50  0000 C CNN
-F 1 "0R05" V 8350 4950 50  0000 C CNN
-F 2 "Resistor_SMD:R_1206_3216Metric" V 8380 4950 50  0001 C CNN
+F 1 "0/0R05" V 8350 4950 50  0000 C CNN
+F 2 "Resistor_SMD:R_0805_2012Metric" V 8380 4950 50  0001 C CNN
 F 3 "~" H 8450 4950 50  0001 C CNN
 	1    8450 4950
@@
 P 8700 5100
 F 0 "C7" H 8815 5146 50  0000 L CNN
-F 1 "100uF" H 8815 5055 50  0000 L CNN
-F 2 "Capacitor_SMD:C_1206_3216Metric" H 8738 4950 50  0001 C CNN
+F 1 "47uF" H 8815 5055 50  0000 L CNN
+F 2 "Capacitor_SMD:C_0805_2012Metric" H 8738 4950 50  0001 C CNN
 F 3 "~" H 8700 5100 50  0001 C CNN
 	1    8700 5100
@@
 	6600 3000 6700 3000
 $Comp
-L Device:Crystal Y1
-U 1 1 5D80BACC
-P 7850 2000
-F 0 "Y1" H 7850 2250 50  0000 C CNN
-F 1 "DNP/32.768kHz" H 7850 2150 50  0000 C CNN
-F 2 "Crystal:Crystal_SMD_TXC_9HT11-2Pin_2.0x1.2mm_HandSoldering" H 7850 2000 50  0001 C CNN
-F 3 "~" H 7850 2000 50  0001 C CNN
-	1    7850 2000
-	1    0    0    -1
-$EndComp
-$Comp
 L Device:Crystal_GND24 Y2
 U 1 1 5D80BAD2
@@
 $EndComp
 Wire Wire Line
-	7700 2000 7600 2000
-Wire Wire Line
-	7600 2000 7600 1700
-Wire Wire Line
-	8000 2000 8100 2000
-Wire Wire Line
 	8400 1800 8400 1700
 Wire Wire Line
@@
 	6600 1400 8400 1400
 Wire Wire Line
-	6600 1700 7600 1700
-Wire Wire Line
 	8900 1300 8900 1700
 Wire Wire Line
 	6600 1300 8900 1300
-Wire Wire Line
-	8100 1600 8100 2000
-Wire Wire Line
-	6600 1600 8100 1600
 $Comp
 L Device:L L4
@@
 	-1   0    0    1
 $EndComp
+NoConn ~ 6600 1600
+NoConn ~ 6600 1700
 $EndSCHEMATC
