File: pcb/usb.sch (KiCad schematic (older format))
At the start: 11 parts, among them J600 USB_B_Micro, U100 LPC5500, U600 USBLC6-2SC6

Commit message: finish sch rev 0.1
Parts:
- removed U100: LPC5500, Package_QFP:TQFP-100-1EP_14x14mm_P0.5mm_EP5x5mm_ThermalVias, symbol symbols:LPC5500
- added U100: LPC5500_FBD64, Package_QFP:LQFP-64-1EP_10x10mm_P0.5mm_EP5x5mm_ThermalVias, symbol symbols:LPC5500_FBD64
Connections:
- net +3V3: now also U100.27 (USB1_3V3), U100.61 (USB0_3V3)
- net GND: now also U100.22 (USB1_VSS), U100.26 (USB1_VSS), U100.64 (USB0_VSS)
- net USB_DM: now also U100.24 (USB1_DM)
- net USB_DP: now also U100.23 (USB1_DP)
- net at R601.2, R602.2: now also U100.25 (USB1_VBUS)
Changed lines of the file:
@@
 EESchema Schematic File Version 4
-LIBS:pcb-cache
 EELAYER 30 0
 EELAYER END
@@
 	-1   0    0    -1
 $EndComp
-$Comp
-L symbols:LPC5500 U100
-U 1 1 5D749DD3
-P 4100 4300
-F 0 "U100" H 4100 4765 50  0000 C CNN
-F 1 "LPC5500" H 4100 4674 50  0000 C CNN
-F 2 "Package_QFP:TQFP-100-1EP_14x14mm_P0.5mm_EP5x5mm_ThermalVias" H 4100 4700 50  0001 C CNN
-F 3 "" H 4000 4350 50  0001 C CNN
-	1    4100 4300
-	1    0    0    -1
-$EndComp
 Wire Wire Line
 	5600 4200 5800 4200
@@
 	4700 4200 5300 4200
 Connection ~ 5300 4200
+$Comp
+L symbols:LPC5500_FBD64 U100
+U 1 1 5EB08D81
+P 4100 4300
+F 0 "U100" H 4100 4765 50  0000 C CNN
+F 1 "LPC5500_FBD64" H 4100 4674 50  0000 C CNN
+F 2 "Package_QFP:LQFP-64-1EP_10x10mm_P0.5mm_EP5x5mm_ThermalVias" H 4100 4700 50  0001 C CNN
+F 3 "" H 4000 4350 50  0001 C CNN
+	1    4100 4300
+	1    0    0    -1
+$EndComp
 $EndSCHEMATC

Commit message: pcb: rev 0.2
Parts:
- removed R608: 1R, Resistor_SMD:R_0603_1608Metric, symbol Device:R
Connections:
- net GND: now also C600.2
Changed lines of the file:
@@
 Wire Wire Line
 	5300 3000 5300 3100
-$Comp
-L Device:R R608
-U 1 1 5D2D5A0B
-P 5300 3550
-F 0 "R608" H 5370 3596 50  0000 L CNN
-F 1 "1R" H 5370 3505 50  0000 L CNN
-F 2 "Resistor_SMD:R_0603_1608Metric" V 5230 3550 50  0001 C CNN
-F 3 "~" H 5300 3550 50  0001 C CNN
-	1    5300 3550
-	-1   0    0    -1
-$EndComp
 Wire Wire Line
 	5600 4200 5800 4200
@@
 L power:GND #PWR0155
 U 1 1 5D76D29D
-P 5300 3700
-F 0 "#PWR0155" H 5300 3450 50  0001 C CNN
-F 1 "GND" H 5305 3527 50  0000 C CNN
-F 2 "" H 5300 3700 50  0001 C CNN
-F 3 "" H 5300 3700 50  0001 C CNN
-	1    5300 3700
+P 5300 3400
+F 0 "#PWR0155" H 5300 3150 50  0001 C CNN
+F 1 "GND" H 5305 3227 50  0000 C CNN
+F 2 "" H 5300 3400 50  0001 C CNN
+F 3 "" H 5300 3400 50  0001 C CNN
+	1    5300 3400
 	-1   0    0    -1
 $EndComp
