File: pcb/audio.sch (KiCad schematic (older format))
At the start: 41 parts, among them J1 AudioJack3_SwitchTR, U400 CS43130, U401 ADP150-3.0, U402 ADP150-1.8, U403 ADP150-1.8, U404 SN74AVC4T245PW, U405 PCA9306, Y400 22.5792MHz

Commit message: finish sch rev 0.1
Parts:
- removed J1: AudioJack3_SwitchTR, footprints:Jack_3.5mm_PJ307C, symbol Connector:AudioJack3_SwitchTR
- removed RV400: RK14J11A0A02, footprints:Potentiometer_RK14J, symbol Device:R_POT
- added C423: 2.2uF, Capacitor_SMD:C_0402_1005Metric, symbol Device:C
- added C424: 1uF, Capacitor_SMD:C_0402_1005Metric, symbol Device:C
- added J1: AudioJack3_SwitchDualS, symbol symbols:AudioJack3_SwitchDualS
- added U406: ADP150-1.8, Package_TO_SOT_SMD:SOT-23-5, symbol Regulator_Linear:AP2112K-1.8
Connections:
- net labels added: +2V0
- net labels removed: ADC1_IN0
- wire segments 132 -> 135
- no-connect marks 3 -> 4
Other:
- moved on the sheet: L401
Changed lines of the file:
@@
 EESchema Schematic File Version 4
-LIBS:pcb-cache
 EELAYER 30 0
 EELAYER END
@@
 Wire Wire Line
 	8900 3400 8600 3400
-Wire Wire Line
-	8600 2500 8600 3400
-Connection ~ 8600 2500
 $Comp
 L Device:C C410
@@
 Wire Wire Line
 	7550 5000 7650 5000
-Wire Wire Line
-	7650 5300 7150 5300
-Wire Wire Line
-	7150 5300 7150 5200
-Wire Wire Line
-	7150 5200 6600 5200
 $Comp
 L power:+1V8 #PWR0267
 U 1 1 5D40EC46
-P 4200 2300
-F 0 "#PWR0267" H 4200 2150 50  0001 C CNN
-F 1 "+1V8" H 4215 2473 50  0000 C CNN
-F 2 "" H 4200 2300 50  0001 C CNN
-F 3 "" H 4200 2300 50  0001 C CNN
-	1    4200 2300
+P 4200 2000
+F 0 "#PWR0267" H 4200 1850 50  0001 C CNN
+F 1 "+1V8" H 4215 2173 50  0000 C CNN
+F 2 "" H 4200 2000 50  0001 C CNN
+F 3 "" H 4200 2000 50  0001 C CNN
+	1    4200 2000
 	1    0    0    -1
 $EndComp
@@
 L Device:L L401
 U 1 1 5D4971D8
-P 4200 2450
-F 0 "L401" H 4253 2496 50  0000 L CNN
-F 1 "120R" H 4253 2405 50  0000 L CNN
-F 2 "Inductor_SMD:L_0603_1608Metric" H 4200 2450 50  0001 C CNN
-F 3 "~" H 4200 2450 50  0001 C CNN
-	1    4200 2450
-	1    0    0    -1
-$EndComp
-$Comp
-L Device:R_POT RV?
-U 1 1 5D1F1382
-P 3500 6800
-AR Path="/5DB51F59/5D1F1382" Ref="RV?"  Part="1"
-AR Path="/5D438133/5D1F1382" Ref="RV400"  Part="1"
-F 0 "RV400" H 3850 6600 50  0000 R CNN
-F 1 "RK14J11A0A02" H 4150 6700 50  0000 R CNN
-F 2 "footprints:Potentiometer_RK14J" H 3500 6800 50  0001 C CNN
-F 3 "~" H 3500 6800 50  0001 C CNN
-	1    3500 6800
-	1    0    0    -1
-$EndComp
-$Comp
-L power:GND #PWR0275
-U 1 1 5D1F4706
-P 3500 7100
-F 0 "#PWR0275" H 3500 6850 50  0001 C CNN
-F 1 "GND" H 3505 6927 50  0000 C CNN
-F 2 "" H 3500 7100 50  0001 C CNN
-F 3 "" H 3500 7100 50  0001 C CNN
-	1    3500 7100
-	1    0    0    -1
-$EndComp
-Wire Wire Line
-	3500 6950 3500 7100
-Wire Wire Line
-	3500 6500 3500 6650
-Text GLabel 4000 6800 2    50   Output ~ 0
-ADC1_IN0
-Wire Wire Line
-	3650 6800 4000 6800
+P 4200 2150
+F 0 "L401" H 4253 2196 50  0000 L CNN
+F 1 "120R" H 4253 2105 50  0000 L CNN
+F 2 "Inductor_SMD:L_0603_1608Metric" H 4200 2150 50  0001 C CNN
+F 3 "~" H 4200 2150 50  0001 C CNN
+	1    4200 2150
+	1    0    0    -1
+$EndComp
 Wire Wire Line
 	5000 5700 4900 5700
 Connection ~ 4900 5700
-$Comp
-L Connector:AudioJack3_SwitchTR J1
-U 1 1 5D440F5D
-P 7850 5100
-F 0 "J1" H 7570 5025 50  0000 R CNN
-F 1 "AudioJack3_SwitchTR" H 7570 4934 50  0000 R CNN
-F 2 "footprints:Jack_3.5mm_PJ307C" H 7850 5100 50  0001 C CNN
-F 3 "~" H 7850 5100 50  0001 C CNN
-	1    7850 5100
-	-1   0    0    -1
-$EndComp
 Wire Wire Line
 	6600 5100 7650 5100
@@
 $EndComp
 $Comp
-L power:+3V3 #PWR?
-U 1 1 5DBD75D1
-P 3500 6500
-F 0 "#PWR?" H 3500 6350 50  0001 C CNN
-F 1 "+3V3" H 3515 6673 50  0000 C CNN
-F 2 "" H 3500 6500 50  0001 C CNN
-F 3 "" H 3500 6500 50  0001 C CNN
-	1    3500 6500
-	1    0    0    -1
-$EndComp
-$Comp
 L Device:Crystal_GND24 Y?
 U 1 1 5DC89C50
@@
 P 2750 2900
 AR Path="/5D4C99F9/5DC89C62" Ref="#PWR?"  Part="1"
-AR Path="/5D438133/5DC89C62" Ref="#PWR?"  Part="1"
-F 0 "#PWR?" H 2750 2650 50  0001 C CNN
+AR Path="/5D438133/5DC89C62" Ref="#PWR0159"  Part="1"
+F 0 "#PWR0159" H 2750 2650 50  0001 C CNN
 F 1 "GND" H 2755 2727 50  0000 C CNN
 F 2 "" H 2750 2900 50  0001 C CNN
@@
 Wire Wire Line
 	3450 2200 2750 2200
+$Comp
+L symbols:+2V0 #PWR0150
+U 1 1 5EA2F5D5
+P 8600 3300
+F 0 "#PWR0150" H 8600 3150 50  0001 C CNN
+F 1 "+2V0" H 8615 3473 50  0000 C CNN
+F 2 "" H 8600 3300 50  0001 C CNN
+F 3 "" H 8600 3300 50  0001 C CNN
+	1    8600 3300
+	1    0    0    -1
+$EndComp
+$Comp
+L power:+3V3 #PWR0160
+U 1 1 5EA302C1
+P 8600 2300
+F 0 "#PWR0160" H 8600 2150 50  0001 C CNN
+F 1 "+3V3" H 8615 2473 50  0000 C CNN
+F 2 "" H 8600 2300 50  0001 C CNN
+F 3 "" H 8600 2300 50  0001 C CNN
+	1    8600 2300
+	1    0    0    -1
+$EndComp
+Wire Wire Line
+	8600 3300 8600 3400
+$Comp
+L Regulator_Linear:AP2112K-1.8 U406
+U 1 1 5EAC96F9
+P 5100 2100
+F 0 "U406" H 5100 2442 50  0000 C CNN
+F 1 "ADP150-1.8" H 5100 2351 50  0000 C CNN
+F 2 "Package_TO_SOT_SMD:SOT-23-5" H 5100 2425 50  0001 C CNN
+F 3 "https://www.diodes.com/assets/Datasheets/AP2112.pdf" H 5100 2200 50  0001 C CNN
+	1    5100 2100
+	-1   0    0    -1
+$EndComp
+Wire Wire Line
+	5500 2000 5400 2000
+Wire Wire Line
+	5400 2100 5500 2100
+Wire Wire Line
+	5500 2100 5500 2000
+Connection ~ 5500 2000
+$Comp
+L power:GND #PWR0161
+U 1 1 5EAC9703
+P 5100 2400
+F 0 "#PWR0161" H 5100 2150 50  0001 C CNN
+F 1 "GND" H 5105 2227 50  0000 C CNN
+F 2 "" H 5100 2400 50  0001 C CNN
+F 3 "" H 5100 2400 50  0001 C CNN
+	1    5100 2400
+	1    0    0    -1
+$EndComp
+$Comp
+L Device:C C424
+U 1 1 5EAC9709
+P 5800 2150
+F 0 "C424" H 5915 2196 50  0000 L CNN
+F 1 "1uF" H 5915 2105 50  0000 L CNN
+F 2 "Capacitor_SMD:C_0402_1005Metric" H 5838 2000 50  0001 C CNN
+F 3 "~" H 5800 2150 50  0001 C CNN
+	1    5800 2150
+	1    0    0    -1
+$EndComp
+$Comp
+L power:GND #PWR0162
+U 1 1 5EAC970F
+P 5800 2300
+F 0 "#PWR0162" H 5800 2050 50  0001 C CNN
+F 1 "GND" H 5805 2127 50  0000 C CNN
+F 2 "" H 5800 2300 50  0001 C CNN
+F 3 "" H 5800 2300 50  0001 C CNN
+	1    5800 2300
+	1    0    0    -1
+$EndComp
+Wire Wire Line
+	5800 2000 5500 2000
+Wire Wire Line
+	4600 2000 4800 2000
+$Comp
+L symbols:+2V0 #PWR0163
+U 1 1 5EAC9719
+P 5500 2000
+F 0 "#PWR0163" H 5500 1850 50  0001 C CNN
+F 1 "+2V0" H 5515 2173 50  0000 C CNN
+F 2 "" H 5500 2000 50  0001 C CNN
+F 3 "" H 5500 2000 50  0001 C CNN
+	1    5500 2000
+	1    0    0    -1
+$EndComp
+$Comp
+L Device:C C423
+U 1 1 5EADB36C
+P 4600 2150
+F 0 "C423" H 4715 2196 50  0000 L CNN
+F 1 "2.2uF" H 4715 2105 50  0000 L CNN
+F 2 "Capacitor_SMD:C_0402_1005Metric" H 4638 2000 50  0001 C CNN
+F 3 "~" H 4600 2150 50  0001 C CNN
+	1    4600 2150
+	1    0    0    -1
+$EndComp
+$Comp
+L power:GND #PWR0164
+U 1 1 5EAEF23D
+P 4600 2300
+F 0 "#PWR0164" H 4600 2050 50  0001 C CNN
+F 1 "GND" H 4605 2127 50  0000 C CNN
+F 2 "" H 4600 2300 50  0001 C CNN
+F 3 "" H 4600 2300 50  0001 C CNN
+	1    4600 2300
+	1    0    0    -1
+$EndComp
+Wire Wire Line
+	4600 2000 4200 2000
+Connection ~ 4600 2000
+Connection ~ 4200 2000
+Wire Wire Line
+	4200 2300 4200 2600
+$Comp
+L symbols:AudioJack3_SwitchDualS J1
+U 1 1 5EB2AE7E
+P 7850 5000
+F 0 "J1" H 7570 4846 50  0000 R CNN
+F 1 "AudioJack3_SwitchDualS" H 7570 4755 50  0000 R CNN
+F 2 "" H 7850 5000 50  0001 C CNN
+F 3 "~" H 7850 5000 50  0001 C CNN
+	1    7850 5000
+	-1   0    0    -1
+$EndComp
+Wire Wire Line
+	6600 5200 7650 5200
+Wire Wire Line
+	7650 5400 6600 5400
+NoConn ~ 7650 5300
 $EndSCHEMATC

Commit message: assign footprints
Parts:
- J1: footprint (none) -> footprints:Jack_3.5mm_PJ327E_5A
Changed lines of the file:
@@
 F 0 "J1" H 7570 4846 50  0000 R CNN
 F 1 "AudioJack3_SwitchDualS" H 7570 4755 50  0000 R CNN
-F 2 "" H 7850 5000 50  0001 C CNN
+F 2 "footprints:Jack_3.5mm_PJ327E_5A" H 7850 5000 50  0001 C CNN
 F 3 "~" H 7850 5000 50  0001 C CNN
 	1    7850 5000

Commit message: rev 0.1
Parts:
- removed C423: 2.2uF, Capacitor_SMD:C_0402_1005Metric, symbol Device:C
- removed L401: 120R, Inductor_SMD:L_0603_1608Metric, symbol Device:L
- removed R404: 10K, Resistor_SMD:R_0603_1608Metric, symbol Device:R
- added C425: 100uF, Capacitor_SMD:C_1206_3216Metric, symbol Device:C
- U401: value ADP150-3.0 -> ADP150-3.3
Connections:
- net +1V8: now also C400.1, C401.1, C402.1, U400.31 (VL), U400.4 (VD)
- net +3V3: no longer C405.1, U401.1 (VIN), U401.3 (EN)
- net GND: now also J1.4, C425.2
- net at U400.22 (HP_DETECT): now also J1.5; no longer J1.4
- new net +SYS: C405.1, C425.1, U401.1 (VIN), U401.3 (EN)
Changed lines of the file:
@@
 P 8200 2500
 F 0 "U401" H 8200 2842 50  0000 C CNN
-F 1 "ADP150-3.0" H 8200 2751 50  0000 C CNN
+F 1 "ADP150-3.3" H 8200 2751 50  0000 C CNN
 F 2 "Package_TO_SOT_SMD:SOT-23-5" H 8200 2825 50  0001 C CNN
 F 3 "https://www.diodes.com/assets/Datasheets/AP2127.pdf" H 8200 2600 50  0001 C CNN
@@
 	6600 5500 7450 5500
 Wire Wire Line
-	7450 5500 7450 5000
-Wire Wire Line
-	7450 5000 7550 5000
-Wire Wire Line
 	6600 5600 7550 5600
 Wire Wire Line
-	7550 5600 7550 5000
+	7550 5600 7550 5400
 Connection ~ 7550 5000
 Wire Wire Line
@@
 Wire Wire Line
 	4900 4600 4900 4800
-$Comp
-L Device:R R404
-U 1 1 5D46D440
-P 4650 5300
-F 0 "R404" V 4600 5100 50  0000 C CNN
-F 1 "10K" V 4600 5500 50  0000 C CNN
-F 2 "Resistor_SMD:R_0603_1608Metric" V 4580 5300 50  0001 C CNN
-F 3 "~" H 4650 5300 50  0001 C CNN
-	1    4650 5300
-	0    1    1    0
-$EndComp
-$Comp
-L power:+1V8 #PWR0271
-U 1 1 5D46FEBD
-P 4300 5300
-F 0 "#PWR0271" H 4300 5150 50  0001 C CNN
-F 1 "+1V8" V 4315 5428 50  0000 L CNN
-F 2 "" H 4300 5300 50  0001 C CNN
-F 3 "" H 4300 5300 50  0001 C CNN
-	1    4300 5300
-	0    -1   -1   0
-$EndComp
-Wire Wire Line
-	4300 5300 4500 5300
-Wire Wire Line
-	4800 5300 5000 5300
 NoConn ~ 5000 3800
 NoConn ~ 5000 3900
@@
 F 3 "" H 3750 2900 50  0001 C CNN
 	1    3750 2900
-	1    0    0    -1
-$EndComp
-$Comp
-L power:GND #PWR0274
-U 1 1 5D490333
-P 3500 3800
-F 0 "#PWR0274" H 3500 3550 50  0001 C CNN
-F 1 "GND" H 3505 3627 50  0000 C CNN
-F 2 "" H 3500 3800 50  0001 C CNN
-F 3 "" H 3500 3800 50  0001 C CNN
-	1    3500 3800
-	1    0    0    -1
-$EndComp
-$Comp
-L Device:L L401
-U 1 1 5D4971D8
-P 4200 2150
-F 0 "L401" H 4253 2196 50  0000 L CNN
-F 1 "120R" H 4253 2105 50  0000 L CNN
-F 2 "Inductor_SMD:L_0603_1608Metric" H 4200 2150 50  0001 C CNN
-F 3 "~" H 4200 2150 50  0001 C CNN
-	1    4200 2150
 	1    0    0    -1
 $EndComp
@@
 	1    0    0    -1
 $EndComp
-$Comp
-L power:+3V3 #PWR0160
-U 1 1 5EA302C1
-P 8600 2300
-F 0 "#PWR0160" H 8600 2150 50  0001 C CNN
-F 1 "+3V3" H 8615 2473 50  0000 C CNN
-F 2 "" H 8600 2300 50  0001 C CNN
-F 3 "" H 8600 2300 50  0001 C CNN
-	1    8600 2300
-	1    0    0    -1
-$EndComp
 Wire Wire Line
 	8600 3300 8600 3400
@@
 Wire Wire Line
 	5800 2000 5500 2000
-Wire Wire Line
-	4600 2000 4800 2000
 $Comp
 L symbols:+2V0 #PWR0163
@@
 	1    0    0    -1
 $EndComp
-$Comp
-L Device:C C423
-U 1 1 5EADB36C
-P 4600 2150
-F 0 "C423" H 4715 2196 50  0000 L CNN
-F 1 "2.2uF" H 4715 2105 50  0000 L CNN
-F 2 "Capacitor_SMD:C_0402_1005Metric" H 4638 2000 50  0001 C CNN
-F 3 "~" H 4600 2150 50  0001 C CNN
-	1    4600 2150
-	1    0    0    -1
-$EndComp
-$Comp
-L power:GND #PWR0164
-U 1 1 5EAEF23D
-P 4600 2300
-F 0 "#PWR0164" H 4600 2050 50  0001 C CNN
-F 1 "GND" H 4605 2127 50  0000 C CNN
-F 2 "" H 4600 2300 50  0001 C CNN
-F 3 "" H 4600 2300 50  0001 C CNN
-	1    4600 2300
-	1    0    0    -1
-$EndComp
-Wire Wire Line
-	4600 2000 4200 2000
-Connection ~ 4600 2000
-Connection ~ 4200 2000
-Wire Wire Line
-	4200 2300 4200 2600
 $Comp
 L symbols:AudioJack3_SwitchDualS J1
@@
 Wire Wire Line
 	6600 5200 7650 5200
-Wire Wire Line
-	7650 5400 6600 5400
-NoConn ~ 7650 5300
+NoConn ~ 5000 5300
+Wire Wire Line
+	7650 5400 7550 5400
+Wire Wire Line
+	7450 5400 7450 5500
+Connection ~ 7550 5400
+Wire Wire Line
+	7550 5400 7550 5000
+Wire Wire Line
+	7550 5400 7450 5400
+Wire Wire Line
+	7650 5300 7350 5300
+Wire Wire Line
+	7350 5300 7350 5400
+Wire Wire Line
+	7350 5400 6600 5400
+$Comp
+L symbols:+SYS #PWR?
+U 1 1 5E8BE692
+P 8600 2300
+AR Path="/5D4C99F9/5E8BE692" Ref="#PWR?"  Part="1"
+AR Path="/5D438133/5E8BE692" Ref="#PWR0114"  Part="1"
+F 0 "#PWR0114" H 8600 2150 50  0001 C CNN
+F 1 "+SYS" H 8615 2473 50  0000 C CNN
+F 2 "" H 8600 2300 50  0001 C CNN
+F 3 "" H 8600 2300 50  0001 C CNN
+	1    8600 2300
+	1    0    0    -1
+$EndComp
+Wire Wire Line
+	4200 2000 4800 2000
+Wire Wire Line
+	4200 2000 4200 2600
+Connection ~ 4200 2000
+Connection ~ 8900 2400
+Wire Wire Line
+	9300 2400 8900 2400
+$Comp
+L power:GND #PWR?
+U 1 1 5EBCBF7D
+P 9300 2700
+AR Path="/5D4C99F9/5EBCBF7D" Ref="#PWR?"  Part="1"
+AR Path="/5D438133/5EBCBF7D" Ref="#PWR0115"  Part="1"
+F 0 "#PWR0115" H 9300 2450 50  0001 C CNN
+F 1 "GND" H 9305 2527 50  0000 C CNN
+F 2 "" H 9300 2700 50  0001 C CNN
+F 3 "" H 9300 2700 50  0001 C CNN
+	1    9300 2700
+	1    0    0    -1
+$EndComp
+$Comp
+L Device:C C?
+U 1 1 5EBCBF77
+P 9300 2550
+AR Path="/5D4C99F9/5EBCBF77" Ref="C?"  Part="1"
+AR Path="/5D438133/5EBCBF77" Ref="C425"  Part="1"
+F 0 "C425" H 9415 2596 50  0000 L CNN
+F 1 "100uF" H 9415 2505 50  0000 L CNN
+F 2 "Capacitor_SMD:C_1206_3216Metric" H 9338 2400 50  0001 C CNN
+F 3 "~" H 9300 2550 50  0001 C CNN
+	1    9300 2550
+	1    0    0    -1
+$EndComp
 $EndSCHEMATC

Commit message: pcb: bug fixes
Parts:
- removed U404: SN74AVC4T245PW, Package_SO:TSSOP-16_4.4x5mm_P0.65mm, symbol Logic_LevelTranslator:SN74AVC4T245PW
- added U404: SN74AVC4T774PW, Package_SO:TSSOP-16_4.4x5mm_P0.65mm, symbol symbols:SN74AVC4T774PW
Connections:
- net +1V8: now also U404.15 (VCCB)
- net +3V3: now also U404.16 (VCCA), U404.2 (DIR2)
- net CODEC_RST: now also U400.28 (~RESET)
- net GND: now also U404.1 (DIR1), U404.10 (GND), U404.7 (DIR3), U404.8 (DIR4), U404.9 (~OE)
- net SAI1_MCLK: now also U404.3 (A1); no longer R400.2
- net SAI1_TXC: now also U404.6 (A4)
- net SAI1_TXD: now also U404.4 (A2)
- net SAI1_TXFS: now also U404.5 (A3)
- net at R401.2: now also U404.13 (B2)
- net at R402.2: now also U404.12 (B3)
- net at R403.2: now also U404.11 (B4)
- new net: R400.2, U404.14 (B1)
Other:
- note added: "DIR L = B to A <-\nDIR H = A to B ->"
- moved on the sheet: C418, C419, R400
Changed lines of the file:
@@
 	1    0    0    -1
 $EndComp
-Text GLabel 1600 4300 0    50   Input ~ 0
+Text GLabel 1600 4300 0    50   Output ~ 0
 SAI1_TXC
-Text GLabel 1600 4200 0    50   Input ~ 0
+Text GLabel 1600 4200 0    50   Output ~ 0
 SAI1_TXFS
 Text GLabel 1600 4100 0    50   Input ~ 0
@@
 Wire Wire Line
 	4100 4300 5000 4300
-Text GLabel 4400 3300 0    50   Output ~ 0
+Text GLabel 1600 4000 0    50   Output ~ 0
 SAI1_MCLK
 $Comp
 L Device:R R400
 U 1 1 5D92452D
-P 4750 3300
-F 0 "R400" V 4700 3100 50  0000 C CNN
-F 1 "33" V 4700 3500 50  0000 C CNN
-F 2 "Resistor_SMD:R_0603_1608Metric" V 4680 3300 50  0001 C CNN
-F 3 "~" H 4750 3300 50  0001 C CNN
-	1    4750 3300
+P 3950 4000
+F 0 "R400" V 3900 3800 50  0000 C CNN
+F 1 "33" V 3900 4200 50  0000 C CNN
+F 2 "Resistor_SMD:R_0603_1608Metric" V 3880 4000 50  0001 C CNN
+F 3 "~" H 3950 4000 50  0001 C CNN
+	1    3950 4000
 	0    1    1    0
 $EndComp
 Wire Wire Line
 	4900 3300 5000 3300
-Wire Wire Line
-	4600 3300 4400 3300
-$Comp
-L Logic_LevelTranslator:SN74AVC4T245PW U404
-U 1 1 5D8C4C20
-P 2500 4000
-F 0 "U404" H 2150 4550 50  0000 C CNN
-F 1 "SN74AVC4T245PW" H 2500 3150 50  0000 C CNN
-F 2 "Package_SO:TSSOP-16_4.4x5mm_P0.65mm" H 2500 3900 50  0001 C CNN
-F 3 "https://www.ti.com/lit/ds/symlink/sn74avc4t245.pdf" H 2450 3750 50  0001 C CNN
-	1    2500 4000
-	1    0    0    -1
-$EndComp
 Wire Wire Line
 	3550 5000 5000 5000
@@
 Wire Wire Line
 	3000 4200 3800 4200
-Wire Wire Line
-	3000 4100 3800 4100
 $Comp
 L Device:R R405
@@
 	3550 4500 3450 4500
 Connection ~ 3450 4500
-Wire Wire Line
-	3000 4400 4800 4400
-Wire Wire Line
-	4800 4400 4800 5200
-Wire Wire Line
-	4800 5200 5000 5200
-Text GLabel 1600 4400 0    50   Input ~ 0
-CODEC_RST
-Wire Wire Line
-	1600 4400 2000 4400
 $Comp
 L power:GND #PWR0121
 U 1 1 5D94B448
-P 2500 4600
-F 0 "#PWR0121" H 2500 4350 50  0001 C CNN
-F 1 "GND" H 2505 4427 50  0000 C CNN
-F 2 "" H 2500 4600 50  0001 C CNN
-F 3 "" H 2500 4600 50  0001 C CNN
-	1    2500 4600
+P 2500 4500
+F 0 "#PWR0121" H 2500 4250 50  0001 C CNN
+F 1 "GND" H 2505 4327 50  0000 C CNN
+F 2 "" H 2500 4500 50  0001 C CNN
+F 3 "" H 2500 4500 50  0001 C CNN
+	1    2500 4500
 	1    0    0    -1
 $EndComp
@@
 Wire Wire Line
 	2600 5000 3000 5000
-Wire Wire Line
-	2000 3600 1900 3600
-Wire Wire Line
-	1900 3600 1900 3700
-Wire Wire Line
-	1900 4600 2500 4600
-Connection ~ 2500 4600
-Wire Wire Line
-	2000 3700 1900 3700
-Connection ~ 1900 3700
-Wire Wire Line
-	1900 3700 1900 4600
-Wire Wire Line
-	2000 3900 1800 3900
-Wire Wire Line
-	1800 3900 1800 3800
-Wire Wire Line
-	1800 3400 2400 3400
-Wire Wire Line
-	2000 3800 1800 3800
-Connection ~ 1800 3800
-Wire Wire Line
-	1800 3800 1800 3400
 $Comp
 L Device:C C418
 U 1 1 5D994C8D
-P 1400 3550
-F 0 "C418" H 1515 3596 50  0000 L CNN
-F 1 "100nF" H 1515 3505 50  0000 L CNN
-F 2 "Capacitor_SMD:C_0402_1005Metric" H 1438 3400 50  0001 C CNN
-F 3 "~" H 1400 3550 50  0001 C CNN
-	1    1400 3550
+P 1400 3450
+F 0 "C418" H 1515 3496 50  0000 L CNN
+F 1 "100nF" H 1515 3405 50  0000 L CNN
+F 2 "Capacitor_SMD:C_0402_1005Metric" H 1438 3300 50  0001 C CNN
+F 3 "~" H 1400 3450 50  0001 C CNN
+	1    1400 3450
 	1    0    0    -1
 $EndComp
@@
 L power:GND #PWR0139
 U 1 1 5D994C93
-P 1400 3700
-F 0 "#PWR0139" H 1400 3450 50  0001 C CNN
-F 1 "GND" H 1405 3527 50  0000 C CNN
-F 2 "" H 1400 3700 50  0001 C CNN
-F 3 "" H 1400 3700 50  0001 C CNN
-	1    1400 3700
+P 1400 3600
+F 0 "#PWR0139" H 1400 3350 50  0001 C CNN
+F 1 "GND" H 1405 3427 50  0000 C CNN
+F 2 "" H 1400 3600 50  0001 C CNN
+F 3 "" H 1400 3600 50  0001 C CNN
+	1    1400 3600
 	1    0    0    -1
 $EndComp
@@
 L power:+3V3 #PWR0140
 U 1 1 5D994C99
-P 1400 3400
-F 0 "#PWR0140" H 1400 3250 50  0001 C CNN
-F 1 "+3V3" H 1415 3573 50  0000 C CNN
-F 2 "" H 1400 3400 50  0001 C CNN
-F 3 "" H 1400 3400 50  0001 C CNN
-	1    1400 3400
-	1    0    0    -1
-$EndComp
-Wire Wire Line
-	1400 3400 1800 3400
-Connection ~ 1400 3400
+P 1400 3300
+F 0 "#PWR0140" H 1400 3150 50  0001 C CNN
+F 1 "+3V3" H 1415 3473 50  0000 C CNN
+F 2 "" H 1400 3300 50  0001 C CNN
+F 3 "" H 1400 3300 50  0001 C CNN
+	1    1400 3300
+	1    0    0    -1
+$EndComp
+Connection ~ 1400 3300
 $Comp
 L power:+1V8 #PWR0142
 U 1 1 5DA41BB7
-P 3000 3400
-F 0 "#PWR0142" H 3000 3250 50  0001 C CNN
-F 1 "+1V8" H 3015 3573 50  0000 C CNN
-F 2 "" H 3000 3400 50  0001 C CNN
-F 3 "" H 3000 3400 50  0001 C CNN
-	1    3000 3400
-	1    0    0    -1
-$EndComp
-Wire Wire Line
-	2600 3400 3000 3400
+P 3000 3300
+F 0 "#PWR0142" H 3000 3150 50  0001 C CNN
+F 1 "+1V8" H 3015 3473 50  0000 C CNN
+F 2 "" H 3000 3300 50  0001 C CNN
+F 3 "" H 3000 3300 50  0001 C CNN
+	1    3000 3300
+	1    0    0    -1
+$EndComp
+Wire Wire Line
+	2600 3300 3000 3300
 $Comp
 L Device:C C419
 U 1 1 5DA47791
-P 3000 3550
-F 0 "C419" H 3115 3596 50  0000 L CNN
-F 1 "100nF" H 3115 3505 50  0000 L CNN
-F 2 "Capacitor_SMD:C_0402_1005Metric" H 3038 3400 50  0001 C CNN
-F 3 "~" H 3000 3550 50  0001 C CNN
-	1    3000 3550
-	1    0    0    -1
-$EndComp
-Connection ~ 3000 3400
+P 3000 3450
+F 0 "C419" H 3115 3496 50  0000 L CNN
+F 1 "100nF" H 3115 3405 50  0000 L CNN
+F 2 "Capacitor_SMD:C_0402_1005Metric" H 3038 3300 50  0001 C CNN
+F 3 "~" H 3000 3450 50  0001 C CNN
+	1    3000 3450
+	1    0    0    -1
+$EndComp
 $Comp
 L power:GND #PWR0143
 U 1 1 5DA4A9B1
-P 3000 3700
-F 0 "#PWR0143" H 3000 3450 50  0001 C CNN
-F 1 "GND" H 3005 3527 50  0000 C CNN
-F 2 "" H 3000 3700 50  0001 C CNN
-F 3 "" H 3000 3700 50  0001 C CNN
-	1    3000 3700
+P 3000 3600
+F 0 "#PWR0143" H 3000 3350 50  0001 C CNN
+F 1 "GND" H 3005 3427 50  0000 C CNN
+F 2 "" H 3000 3600 50  0001 C CNN
+F 3 "" H 3000 3600 50  0001 C CNN
+	1    3000 3600
 	1    0    0    -1
 $EndComp
@@
 	1    0    0    -1
 $EndComp
+Connection ~ 3000 3300
+Text GLabel 4600 5200 0    50   Input ~ 0
+CODEC_RST
+$Comp
+L symbols:SN74AVC4T774PW U404
+U 1 1 5E85A42F
+P 2500 3900
+F 0 "U404" H 2800 3350 50  0000 C CNN
+F 1 "SN74AVC4T774PW" H 2900 3250 50  0000 C CNN
+F 2 "Package_SO:TSSOP-16_4.4x5mm_P0.65mm" H 2500 3800 50  0001 C CNN
+F 3 "https://www.ti.com/lit/ds/symlink/sn74avc4t245.pdf" H 2450 3650 50  0001 C CNN
+	1    2500 3900
+	1    0    0    -1
+$EndComp
+Wire Wire Line
+	4600 5200 5000 5200
+Wire Wire Line
+	3000 4100 3800 4100
+Wire Wire Line
+	2000 4000 1600 4000
+Wire Wire Line
+	4100 4000 4900 4000
+Wire Wire Line
+	4900 4000 4900 3300
+Wire Wire Line
+	3000 4000 3800 4000
+Wire Wire Line
+	1400 3300 1800 3300
+Wire Wire Line
+	2000 3900 1900 3900
+Wire Wire Line
+	1900 3900 1900 4500
+Wire Wire Line
+	1900 4500 2500 4500
+Connection ~ 2500 4500
+Text Notes 1850 3250 0    50   ~ 0
+DIR L = B to A <-\nDIR H = A to B ->
+Wire Wire Line
+	2000 3500 1900 3500
+Wire Wire Line
+	1900 3500 1900 3700
+Connection ~ 1900 3900
+Wire Wire Line
+	2000 3700 1900 3700
+Connection ~ 1900 3700
+Wire Wire Line
+	1900 3700 1900 3800
+Wire Wire Line
+	2000 3800 1900 3800
+Connection ~ 1900 3800
+Wire Wire Line
+	1900 3800 1900 3900
+Wire Wire Line
+	2000 3600 1800 3600
+Wire Wire Line
+	1800 3600 1800 3300
+Connection ~ 1800 3300
+Wire Wire Line
+	1800 3300 2400 3300
 $EndSCHEMATC
