File: pcb/audio.sch (KiCad schematic (older format))
At the start: 41 parts, among them J1 AudioJack3_SwitchDualS, U400 CS43130, U401 ADP150-3.3, U402 ADP150-1.8, U403 ADP150-1.8, U404 SN74AVC4T774PW, U405 PCA9306, U406 ADP150-1.8, Y400 22.5792MHz

Commit message: pcb: rev 0.2
Parts:
- C404: value 4.7uF -> 10uF
- C425: value 100uF -> 47uF; footprint Capacitor_SMD:C_1206_3216Metric -> Capacitor_SMD:C_0805_2012Metric
- R400, R401, R402, R403: footprint Resistor_SMD:R_0603_1608Metric -> Resistor_SMD:R_0402_1005Metric
- R407: value 200K -> 100K
Connections:
- net +3V3: now also U404.8 (DIR4); no longer U404.2 (DIR2)
- net GND: now also U404.2 (DIR2); no longer U404.8 (DIR4)
- net SAI1_TXC: now also U404.4 (A2); no longer U404.6 (A4)
- net SAI1_TXD: now also U404.6 (A4); no longer U404.4 (A2)
- net at U400.2 (SDIN1): now also R403.1; no longer R401.1
- net at U400.34 (SCLK1): now also R401.1; no longer R403.1
Changed lines of the file:
@@
 P 7600 2550
 F 0 "C404" H 7715 2596 50  0000 L CNN
-F 1 "4.7uF" H 7715 2505 50  0000 L CNN
+F 1 "10uF" H 7715 2505 50  0000 L CNN
 F 2 "Capacitor_SMD:C_0603_1608Metric" H 7638 2400 50  0001 C CNN
 F 3 "~" H 7600 2550 50  0001 C CNN
@@
 F 0 "R401" V 3900 3900 50  0000 C CNN
 F 1 "33" V 3900 4300 50  0000 C CNN
-F 2 "Resistor_SMD:R_0603_1608Metric" V 3880 4100 50  0001 C CNN
+F 2 "Resistor_SMD:R_0402_1005Metric" V 3880 4100 50  0001 C CNN
 F 3 "~" H 3950 4100 50  0001 C CNN
 	1    3950 4100
@@
 F 0 "R402" V 3900 4000 50  0000 C CNN
 F 1 "33" V 3900 4400 50  0000 C CNN
-F 2 "Resistor_SMD:R_0603_1608Metric" V 3880 4200 50  0001 C CNN
+F 2 "Resistor_SMD:R_0402_1005Metric" V 3880 4200 50  0001 C CNN
 F 3 "~" H 3950 4200 50  0001 C CNN
 	1    3950 4200
@@
 F 0 "R403" V 3900 4100 50  0000 C CNN
 F 1 "33" V 3900 4500 50  0000 C CNN
-F 2 "Resistor_SMD:R_0603_1608Metric" V 3880 4300 50  0001 C CNN
+F 2 "Resistor_SMD:R_0402_1005Metric" V 3880 4300 50  0001 C CNN
 F 3 "~" H 3950 4300 50  0001 C CNN
 	1    3950 4300
@@
 	1    0    0    -1
 $EndComp
-Text GLabel 1600 4300 0    50   Output ~ 0
+Text GLabel 1600 4100 0    50   Output ~ 0
 SAI1_TXC
 Text GLabel 1600 4200 0    50   Output ~ 0
 SAI1_TXFS
-Text GLabel 1600 4100 0    50   Input ~ 0
+Text GLabel 1600 4300 0    50   Input ~ 0
 SAI1_TXD
 Text GLabel 1700 5500 0    50   Input ~ 0
@@
 I2C1_SDA
 Wire Wire Line
+	1600 4300 2000 4300
+Wire Wire Line
+	1600 4200 2000 4200
+Wire Wire Line
 	1600 4100 2000 4100
 Wire Wire Line
-	1600 4200 2000 4200
-Wire Wire Line
-	1600 4300 2000 4300
-Wire Wire Line
-	4100 4100 5000 4100
-Wire Wire Line
 	4100 4200 5000 4200
-Wire Wire Line
-	4100 4300 5000 4300
 Text GLabel 1600 4000 0    50   Output ~ 0
 SAI1_MCLK
@@
 F 0 "R400" V 3900 3800 50  0000 C CNN
 F 1 "33" V 3900 4200 50  0000 C CNN
-F 2 "Resistor_SMD:R_0603_1608Metric" V 3880 4000 50  0001 C CNN
+F 2 "Resistor_SMD:R_0402_1005Metric" V 3880 4000 50  0001 C CNN
 F 3 "~" H 3950 4000 50  0001 C CNN
 	1    3950 4000
@@
 P 1900 5250
 F 0 "R407" H 1750 5100 50  0000 C CNN
-F 1 "200K" H 1750 5200 50  0000 C CNN
+F 1 "100K" H 1750 5200 50  0000 C CNN
 F 2 "Resistor_SMD:R_0603_1608Metric" V 1830 5250 50  0001 C CNN
 F 3 "~" H 1900 5250 50  0001 C CNN
@@
 AR Path="/5D438133/5EBCBF77" Ref="C425"  Part="1"
 F 0 "C425" H 9415 2596 50  0000 L CNN
-F 1 "100uF" H 9415 2505 50  0000 L CNN
-F 2 "Capacitor_SMD:C_1206_3216Metric" H 9338 2400 50  0001 C CNN
+F 1 "47uF" H 9415 2505 50  0000 L CNN
+F 2 "Capacitor_SMD:C_0805_2012Metric" H 9338 2400 50  0001 C CNN
 F 3 "~" H 9300 2550 50  0001 C CNN
 	1    9300 2550
@@
 	2000 3500 1900 3500
 Wire Wire Line
-	1900 3500 1900 3700
+	1900 3500 1900 3600
 Connection ~ 1900 3900
 Wire Wire Line
 	2000 3700 1900 3700
 Connection ~ 1900 3700
-Wire Wire Line
-	1900 3700 1900 3800
-Wire Wire Line
-	2000 3800 1900 3800
-Connection ~ 1900 3800
-Wire Wire Line
-	1900 3800 1900 3900
-Wire Wire Line
-	2000 3600 1800 3600
-Wire Wire Line
-	1800 3600 1800 3300
 Connection ~ 1800 3300
 Wire Wire Line
 	1800 3300 2400 3300
+Wire Wire Line
+	4500 4100 4500 4300
+Wire Wire Line
+	4500 4300 4100 4300
+Wire Wire Line
+	4500 4100 5000 4100
+Wire Wire Line
+	4100 4100 4400 4100
+Wire Wire Line
+	4400 4100 4400 4400
+Wire Wire Line
+	4400 4400 4600 4400
+Wire Wire Line
+	4600 4400 4600 4300
+Wire Wire Line
+	4600 4300 5000 4300
+Wire Wire Line
+	1900 3700 1900 3900
+Wire Wire Line
+	2000 3600 1900 3600
+Connection ~ 1900 3600
+Wire Wire Line
+	1900 3600 1900 3700
+Wire Wire Line
+	1800 3800 2000 3800
+Wire Wire Line
+	1800 3300 1800 3800
 $EndSCHEMATC

Commit message: pcb: rev 0.3
Parts:
- added C426: 47uF, Capacitor_SMD:C_0805_2012Metric, symbol Device:C
Connections:
- net +2V0: now also C426.1
- net +3V3: now also C420.2; no longer C420.1
- net GND: now also C420.1, C426.2; no longer C420.2
Changed lines of the file:
@@
 F 3 "~" H 1500 5150 50  0001 C CNN
 	1    1500 5150
-	1    0    0    -1
+	1    0    0    1
 $EndComp
 Connection ~ 1500 5000
@@
 Wire Wire Line
 	1800 3300 1800 3800
+$Comp
+L power:GND #PWR?
+U 1 1 5F264DFE
+P 9300 3700
+AR Path="/5D4C99F9/5F264DFE" Ref="#PWR?"  Part="1"
+AR Path="/5D438133/5F264DFE" Ref="#PWR0106"  Part="1"
+F 0 "#PWR0106" H 9300 3450 50  0001 C CNN
+F 1 "GND" H 9305 3527 50  0000 C CNN
+F 2 "" H 9300 3700 50  0001 C CNN
+F 3 "" H 9300 3700 50  0001 C CNN
+	1    9300 3700
+	1    0    0    -1
+$EndComp
+$Comp
+L Device:C C?
+U 1 1 5F264E04
+P 9300 3550
+AR Path="/5D4C99F9/5F264E04" Ref="C?"  Part="1"
+AR Path="/5D438133/5F264E04" Ref="C426"  Part="1"
+F 0 "C426" H 9415 3596 50  0000 L CNN
+F 1 "47uF" H 9415 3505 50  0000 L CNN
+F 2 "Capacitor_SMD:C_0805_2012Metric" H 9338 3400 50  0001 C CNN
+F 3 "~" H 9300 3550 50  0001 C CNN
+	1    9300 3550
+	1    0    0    -1
+$EndComp
+Wire Wire Line
+	9300 3400 8900 3400
+Connection ~ 8900 3400
 $EndSCHEMATC
