File: pcb/lcd.sch (KiCad schematic (older format))
At the start: 33 parts, among them J500 FPC_18P_1.0MM, U501 LT1617, U502 LM324

Commit message: finish sch rev 0.1
Parts:
- removed J500: FPC_18P_1.0MM, Connector_FFC-FPC:TE_1-84953-8_1x18-1MP_P1.0mm_Horizontal, symbol Connector_Generic:Conn_01x18
- removed L501: 22uH, Inductor_SMD:L_Vishay_IHLP-1212, symbol Device:L
- removed R503: 330K, Resistor_SMD:R_0603_1608Metric, symbol Device:R
- removed R505, R507, R508: 10K, Resistor_SMD:R_0603_1608Metric, symbol Device:R
- removed R506: 75K, Resistor_SMD:R_0603_1608Metric, symbol Device:R
- removed R509: 20K, Resistor_SMD:R_0603_1608Metric, symbol Device:R
- removed R510, R511, R512, R513, R514: 33, Resistor_SMD:R_0603_1608Metric, symbol Device:R
- removed RN502: 33R, Resistor_SMD:R_Array_Convex_4x0402, symbol Device:R_Pack04
- removed RV500: RK14J11A0A02/50K, footprints:Potentiometer_RK14J, symbol Device:R_POT
- removed U501: LT1617, Package_TO_SOT_SMD:TSOT-23-5, symbol symbols:LT1617
- removed U502: LM324, Package_SO:TSSOP-14_4.4x5mm_P0.65mm, symbol Amplifier_Operational:LM324
- added C513: 4.7uF/25V, Capacitor_SMD:C_0603_1608Metric, symbol Device:C
- added D502, D503: MBR0530, Diode_SMD:D_SOD-123, symbol Device:D_Schottky
- added J500: FPC_24P_0.5MM, Connector_FFC-FPC:Hirose_FH12-24S-0.5SH_1x24-1MP_P0.50mm_Horizontal, symbol Connector_Generic:Conn_01x24
- added Q?: Q_NMOS_GSD, Package_TO_SOT_SMD:SOT-323_SC-70, symbol Device:Q_NMOS_GSD
- added R502: 10K, Resistor_SMD:R_0603_1608Metric, symbol Device:R
- C501, C509: value 22uF/25V -> 4.7uF/25V
- C502, C506, C507: value 4.7uF -> 4.7uF/25V
- C504, C505: value 4.7uF -> 1uF
- C508: value 10uF -> 4.7uF/25V
- C510: value 220nF -> 1uF
- L500: value 22uH -> 10uH
- R503: renamed from R504; value 10K -> 3R
Connections:
- net labels added: EPD_BUSY, EPD_CS, EPD_DC, EPD_RST, EPD_SCLK, EPD_SDI, GDR, POR, PREVGH, PREVGL, RESE, SPI_MOSI, SPI_SCK, SPI_SSEL0
- net labels removed: LCD_CP, LCD_CPG, LCD_CPL, LCD_D0, LCD_D1, LCD_FR, LCD_S, LCD_ST, LCD_V1, LCD_V2, LCD_V3, LCD_V4, LCD_V5, STN_CP, STN_CPG, STN_CPL, STN_D0, STN_D1, STN_FR, STN_S, STN_ST, ~LCD_PWR_EN
- wire segments 118 -> 63
- no-connect marks 0 -> 3
Other:
- note removed: "-7V to -22V"
- moved on the sheet: C501, C502, C503, C504, C505, C506, C507, C508, C509, C510, C512, D501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

Commit message: assign footprints
Parts:
- C501, C509: footprint Capacitor_SMD:C_1206_3216Metric -> Capacitor_SMD:C_0805_2012Metric
- C502, C506, C507, C508, C512, C513: footprint Capacitor_SMD:C_0603_1608Metric -> Capacitor_SMD:C_0805_2012Metric
- gave numbers to parts that had none: 1
Changed lines of the file:
@@
 F 0 "C508" V 7200 4700 50  0000 C CNN
 F 1 "4.7uF/25V" V 7200 5150 50  0000 C CNN
-F 2 "Capacitor_SMD:C_0603_1608Metric" H 7288 4750 50  0001 C CNN
+F 2 "Capacitor_SMD:C_0805_2012Metric" H 7288 4750 50  0001 C CNN
 F 3 "~" H 7250 4900 50  0001 C CNN
 	1    7250 4900
@@
 F 0 "C512" H 3385 3604 50  0000 R CNN
 F 1 "4.7uF/25V" H 3385 3695 50  0000 R CNN
-F 2 "Capacitor_SMD:C_0603_1608Metric" H 3538 3500 50  0001 C CNN
+F 2 "Capacitor_SMD:C_0805_2012Metric" H 3538 3500 50  0001 C CNN
 F 3 "~" H 3500 3650 50  0001 C CNN
 	1    3500 3650
@@
 F 0 "C506" V 7300 5000 50  0000 R CNN
 F 1 "4.7uF/25V" V 7300 4650 50  0000 R CNN
-F 2 "Capacitor_SMD:C_0603_1608Metric" H 7288 4550 50  0001 C CNN
+F 2 "Capacitor_SMD:C_0805_2012Metric" H 7288 4550 50  0001 C CNN
 F 3 "~" H 7250 4700 50  0001 C CNN
 	1    7250 4700
@@
 F 0 "C507" V 7300 5100 50  0000 R CNN
 F 1 "4.7uF/25V" V 7300 5550 50  0000 R CNN
-F 2 "Capacitor_SMD:C_0603_1608Metric" H 7288 4650 50  0001 C CNN
+F 2 "Capacitor_SMD:C_0805_2012Metric" H 7288 4650 50  0001 C CNN
 F 3 "~" H 7250 4800 50  0001 C CNN
 	1    7250 4800
@@
 F 0 "C502" V 7300 3500 50  0000 R CNN
 F 1 "4.7uF/25V" V 7300 3150 50  0000 R CNN
-F 2 "Capacitor_SMD:C_0603_1608Metric" H 7288 3050 50  0001 C CNN
+F 2 "Capacitor_SMD:C_0805_2012Metric" H 7288 3050 50  0001 C CNN
 F 3 "~" H 7250 3200 50  0001 C CNN
 	1    7250 3200
@@
 F 0 "C509" V 7200 4700 50  0000 L CNN
 F 1 "4.7uF/25V" V 7200 4250 50  0000 L CNN
-F 2 "Capacitor_SMD:C_1206_3216Metric" H 7288 4850 50  0001 C CNN
+F 2 "Capacitor_SMD:C_0805_2012Metric" H 7288 4850 50  0001 C CNN
 F 3 "~" H 7250 5000 50  0001 C CNN
 	1    7250 5000
@@
 F 0 "C501" V 7300 3200 50  0000 L CNN
 F 1 "4.7uF/25V" V 7300 2650 50  0000 L CNN
-F 2 "Capacitor_SMD:C_1206_3216Metric" H 7288 2950 50  0001 C CNN
+F 2 "Capacitor_SMD:C_0805_2012Metric" H 7288 2950 50  0001 C CNN
 F 3 "~" H 7250 3100 50  0001 C CNN
 	1    7250 3100
@@
 $EndComp
 $Comp
-L Device:Q_NMOS_GSD Q?
+L Device:Q_NMOS_GSD Q1
 U 1 1 5EBD17BB
 P 4100 3800
-F 0 "Q?" H 4304 3846 50  0000 L CNN
+F 0 "Q1" H 4304 3846 50  0000 L CNN
 F 1 "Q_NMOS_GSD" H 4304 3755 50  0000 L CNN
 F 2 "Package_TO_SOT_SMD:SOT-323_SC-70" H 4300 3900 50  0001 C CNN
@@
 F 0 "C513" H 4085 3304 50  0000 R CNN
 F 1 "4.7uF/25V" H 4085 3395 50  0000 R CNN
-F 2 "Capacitor_SMD:C_0603_1608Metric" H 4238 3200 50  0001 C CNN
+F 2 "Capacitor_SMD:C_0805_2012Metric" H 4238 3200 50  0001 C CNN
 F 3 "~" H 4200 3350 50  0001 C CNN
 	1    4200 3350

Commit message: rev 0.1
Parts:
- J500: value FPC_24P_0.5MM -> FH12A-24S-0.5SH
Connections:
- net labels added: EPD_RS
Changed lines of the file:
@@
 P 7900 3900
 F 0 "J500" H 7980 3892 50  0000 L CNN
-F 1 "FPC_24P_0.5MM" H 7980 3801 50  0000 L CNN
+F 1 "FH12A-24S-0.5SH" H 7980 3801 50  0000 L CNN
 F 2 "Connector_FFC-FPC:Hirose_FH12-24S-0.5SH_1x24-1MP_P0.50mm_Horizontal" H 7900 3900 50  0001 C CNN
 F 3 "~" H 7900 3900 50  0001 C CNN
@@
 EPD_RST
 Text Label 7100 3800 0    50   ~ 0
-EPD_DC
+EPD_RS
 Text Label 7100 3900 0    50   ~ 0
 EPD_CS

Commit message: pcb: bug fixes
Parts:
- removed C501: 4.7uF/25V, Capacitor_SMD:C_0805_2012Metric, symbol Device:C
- removed C505: 1uF, Capacitor_SMD:C_0603_1608Metric, symbol Device:C
- D501, D502, D503: value MBR0530 -> NSR0530H; footprint Diode_SMD:D_SOD-123 -> Diode_SMD:D_SOD-323
- J500: footprint Connector_FFC-FPC:Hirose_FH12-24S-0.5SH_1x24-1MP_P0.50mm_Horizontal -> footprints:Hirose_FH12A-24S-0.5SH_1x24-1MP_P0.50mm_Horizontal
Connections:
- net labels removed: POR
- wire segments 63 -> 57
Changed lines of the file:
@@
 P 4650 3500
 F 0 "D501" H 4850 3450 50  0000 C CNN
-F 1 "MBR0530" H 4400 3450 50  0000 C CNN
-F 2 "Diode_SMD:D_SOD-123" H 4650 3500 50  0001 C CNN
+F 1 "NSR0530H" H 4400 3450 50  0000 C CNN
+F 2 "Diode_SMD:D_SOD-323" H 4650 3500 50  0001 C CNN
 F 3 "~" H 4650 3500 50  0001 C CNN
 	1    4650 3500
@@
 $EndComp
 $Comp
-L Device:C C505
-U 1 1 5DB2BE84
-P 7250 4600
-F 0 "C505" V 7300 4900 50  0000 R CNN
-F 1 "1uF" V 7300 4500 50  0000 R CNN
-F 2 "Capacitor_SMD:C_0603_1608Metric" H 7288 4450 50  0001 C CNN
-F 3 "~" H 7250 4600 50  0001 C CNN
-	1    7250 4600
-	0    -1   -1   0
-$EndComp
-$Comp
 L Device:C C506
 U 1 1 5DB2C2C4
@@
 $EndComp
 $Comp
-L Device:C C?
-U 1 1 5DB8753F
-P 7250 3100
-AR Path="/5D4C99F9/5DB8753F" Ref="C?"  Part="1"
-AR Path="/5DB51F59/5DB8753F" Ref="C501"  Part="1"
-F 0 "C501" V 7300 3200 50  0000 L CNN
-F 1 "4.7uF/25V" V 7300 2650 50  0000 L CNN
-F 2 "Capacitor_SMD:C_0805_2012Metric" H 7288 2950 50  0001 C CNN
-F 3 "~" H 7250 3100 50  0001 C CNN
-	1    7250 3100
-	0    -1   -1   0
-$EndComp
-$Comp
 L Connector_Generic:Conn_01x24 J500
 U 1 1 5EB57FB2
@@
 F 0 "J500" H 7980 3892 50  0000 L CNN
 F 1 "FH12A-24S-0.5SH" H 7980 3801 50  0000 L CNN
-F 2 "Connector_FFC-FPC:Hirose_FH12-24S-0.5SH_1x24-1MP_P0.50mm_Horizontal" H 7900 3900 50  0001 C CNN
+F 2 "footprints:Hirose_FH12A-24S-0.5SH_1x24-1MP_P0.50mm_Horizontal" H 7900 3900 50  0001 C CNN
 F 3 "~" H 7900 3900 50  0001 C CNN
 	1    7900 3900
@@
 	7000 4700 7000 4800
 Connection ~ 7000 4800
-Wire Wire Line
-	7100 4600 7000 4600
-Wire Wire Line
-	7000 4600 7000 4700
 Connection ~ 7000 4700
 Wire Wire Line
 	7100 4500 7000 4500
-Wire Wire Line
-	7000 4500 7000 4600
-Connection ~ 7000 4600
 Wire Wire Line
 	7700 4400 7000 4400
@@
 	7400 4500 7700 4500
 Wire Wire Line
-	7400 4600 7700 4600
-Wire Wire Line
 	7400 4700 7700 4700
 Wire Wire Line
@@
 Connection ~ 7000 4400
 Wire Wire Line
-	7400 3100 7700 3100
-Wire Wire Line
 	7400 3200 7700 3200
-Wire Wire Line
-	7100 3100 7000 3100
-Wire Wire Line
-	7000 3100 7000 3200
 Connection ~ 7000 4200
 Wire Wire Line
 	7100 3200 7000 3200
-Connection ~ 7000 3200
 $Comp
 L Device:R R502
@@
 EPD_BUSY
 Text GLabel 6200 3700 0    50   Input ~ 0
-POR
+EPD_RST
 Text GLabel 6200 3800 0    50   Input ~ 0
 EPD_DC
@@
 P 4650 2900
 F 0 "D503" H 4450 2950 50  0000 C CNN
-F 1 "MBR0530" H 4900 2950 50  0000 C CNN
-F 2 "Diode_SMD:D_SOD-123" H 4650 2900 50  0001 C CNN
+F 1 "NSR0530H" H 4900 2950 50  0000 C CNN
+F 2 "Diode_SMD:D_SOD-323" H 4650 2900 50  0001 C CNN
 F 3 "~" H 4650 2900 50  0001 C CNN
 	1    4650 2900
@@
 P 4650 3200
 F 0 "D502" H 4850 3150 50  0000 C CNN
-F 1 "MBR0530" H 4400 3150 50  0000 C CNN
-F 2 "Diode_SMD:D_SOD-123" H 4650 3200 50  0001 C CNN
+F 1 "NSR0530H" H 4400 3150 50  0000 C CNN
+F 2 "Diode_SMD:D_SOD-323" H 4650 3200 50  0001 C CNN
 F 3 "~" H 4650 3200 50  0001 C CNN
 	1    4650 3200
@@
 Text Label 7400 5000 0    50   ~ 0
 PREVGL
+Wire Wire Line
+	7000 4500 7000 4700
 $EndSCHEMATC

Commit message: pcb: rev 0.3
Connections:
- wire segments 57 -> 58
Changed lines of the file:
@@
 Wire Wire Line
 	7000 4500 7000 4700
+Text Label 4300 4000 0    50   ~ 0
+RESE
+Wire Wire Line
+	4200 4000 4800 4000
+Connection ~ 4200 4000
 $EndSCHEMATC
