File: pcb/storage.sch (KiCad schematic (older format))
At the start: 11 parts, among them Q300 IRLML6402

Commit message: rev 0.1
Parts:
- R301, R302, R303: footprint Resistor_SMD:R_0603_1608Metric -> Resistor_SMD:R_0402_1005Metric
Changed lines of the file:
@@
 F 0 "R301" H 6470 2996 50  0000 L CNN
 F 1 "10K" H 6470 2905 50  0000 L CNN
-F 2 "Resistor_SMD:R_0603_1608Metric" V 6330 2950 50  0001 C CNN
+F 2 "Resistor_SMD:R_0402_1005Metric" V 6330 2950 50  0001 C CNN
 F 3 "~" H 6400 2950 50  0001 C CNN
 	1    6400 2950
@@
 F 0 "R302" H 5970 2996 50  0000 L CNN
 F 1 "10K" H 5970 2905 50  0000 L CNN
-F 2 "Resistor_SMD:R_0603_1608Metric" V 5830 2950 50  0001 C CNN
+F 2 "Resistor_SMD:R_0402_1005Metric" V 5830 2950 50  0001 C CNN
 F 3 "~" H 5900 2950 50  0001 C CNN
 	1    5900 2950
@@
 F 0 "R303" V 6600 3300 50  0000 C CNN
 F 1 "33R" V 6600 3700 50  0000 C CNN
-F 2 "Resistor_SMD:R_0603_1608Metric" V 6580 3500 50  0001 C CNN
+F 2 "Resistor_SMD:R_0402_1005Metric" V 6580 3500 50  0001 C CNN
 F 3 "~" H 6650 3500 50  0001 C CNN
 	1    6650 3500

Commit message: pcb: rev 0.2
Parts:
- removed D300: RB521S30T1G, Diode_SMD:D_SOD-523, symbol Device:D_Schottky
- added Q301: BSS138, Package_TO_SOT_SMD:SOT-23, symbol Transistor_FET:BSS138
- added R306, R307, R308: 47K, Resistor_SMD:R_0402_1005Metric, symbol Device:R
- Q300: value IRLML6402 -> PMV48XP
- R301, R302: value 10K -> 47K
- R305: value 10K -> 47K; footprint Resistor_SMD:R_0603_1608Metric -> Resistor_SMD:R_0402_1005Metric
Connections:
- net +3V3: no longer R302.1
- net GND: now also Q301.2 (S); no longer R305.2
- net SD0_CMD: now also R307.2; no longer R302.2
- net SD0_D0: now also R306.2
- net SD0_D1: now also R305.2
- net SD0_D2: now also R302.2
- net SD0_D3: now also R308.2
- net at Q300.1 (G), R304.2: now also Q301.3 (D); no longer R305.1
- net +VSD: now reaches C301.1, C302.1, MICRO_SD300.4 (VDD), Q300.3 (D)
- net +VSD: now also R302.1, R305.1, R306.1, R307.1, R308.1
- new net SD0_PWR_EN: Q301.1 (G)
Other:
- moved on the sheet: C301, C302, Q300, R301, R303, R304

Commit message: pcb: rev 0.3
Parts:
- removed Q300: PMV48XP, Package_TO_SOT_SMD:SOT-23, symbol Transistor_FET:IRLML6402
- removed Q301: BSS138, Package_TO_SOT_SMD:SOT-23, symbol Transistor_FET:BSS138
- removed R304: 100K, Resistor_SMD:R_0603_1608Metric, symbol Device:R
Connections:
- net +VSD is gone; now on net +3V3: C301.1, C302.1, MICRO_SD300.4 (VDD), R302.1, R305.1, R306.1, R307.1, R308.1
Changed lines of the file:
@@
 	8000 3000 7600 3000
 Connection ~ 7600 3000
-$Comp
-L power:+3V3 #PWR0203
-U 1 1 5D1E3230
-P 5900 1800
-F 0 "#PWR0203" H 5900 1650 50  0001 C CNN
-F 1 "+3V3" H 5915 1973 50  0000 C CNN
-F 2 "" H 5900 1800 50  0001 C CNN
-F 3 "" H 5900 1800 50  0001 C CNN
-	1    5900 1800
-	1    0    0    -1
-$EndComp
-$Comp
-L Transistor_FET:IRLML6402 Q300
-U 1 1 5D1E5978
-P 5800 2100
-F 0 "Q300" H 6006 2054 50  0000 L CNN
-F 1 "PMV48XP" H 6006 2145 50  0000 L CNN
-F 2 "Package_TO_SOT_SMD:SOT-23" H 6000 2025 50  0001 L CIN
-F 3 "https://www.infineon.com/dgdl/irlml6402pbf.pdf?fileId=5546d462533600a401535668d5c2263c" H 5800 2100 50  0001 L CNN
-	1    5800 2100
-	1    0    0    1
-$EndComp
-Wire Wire Line
-	5900 1800 5900 1900
-$Comp
-L Device:R R304
-U 1 1 5D1FF47A
-P 5450 1950
-F 0 "R304" H 5520 1996 50  0000 L CNN
-F 1 "100K" H 5520 1905 50  0000 L CNN
-F 2 "Resistor_SMD:R_0603_1608Metric" V 5380 1950 50  0001 C CNN
-F 3 "~" H 5450 1950 50  0001 C CNN
-	1    5450 1950
-	1    0    0    -1
-$EndComp
-Text GLabel 4700 3200 0    50   Input ~ 0
-SD0_PWR_EN
-Wire Wire Line
-	5900 2300 5900 2700
-$Comp
-L power:+3V3 #PWR0205
-U 1 1 5D20B20B
-P 5450 1800
-F 0 "#PWR0205" H 5450 1650 50  0001 C CNN
-F 1 "+3V3" H 5465 1973 50  0000 C CNN
-F 2 "" H 5450 1800 50  0001 C CNN
-F 3 "" H 5450 1800 50  0001 C CNN
-	1    5450 1800
-	1    0    0    -1
-$EndComp
 Text Notes 7800 3100 0    50   ~ 0
 47uF is required to comply with SD 3.0 spec
@@
 	1    0    0    -1
 $EndComp
-Text Label 5000 3200 0    50   ~ 0
-SD_PWR_EN
 Text Label 5000 3700 0    50   ~ 0
 SD_CLK
@@
 Wire Wire Line
 	4700 3900 5600 3900
-$Comp
-L Transistor_FET:BSS138 Q301
-U 1 1 5E8D0007
-P 5350 2300
-F 0 "Q301" H 5554 2346 50  0000 L CNN
-F 1 "BSS138" H 5554 2255 50  0000 L CNN
-F 2 "Package_TO_SOT_SMD:SOT-23" H 5550 2225 50  0001 L CIN
-F 3 "https://www.fairchildsemi.com/datasheets/BS/BSS138.pdf" H 5350 2300 50  0001 L CNN
-	1    5350 2300
-	1    0    0    -1
-$EndComp
-Wire Wire Line
-	5600 2100 5450 2100
-Connection ~ 5450 2100
-Wire Wire Line
-	4700 3200 5100 3200
-$Comp
-L power:GND #PWR0106
-U 1 1 5E8F5B98
-P 5450 2500
-F 0 "#PWR0106" H 5450 2250 50  0001 C CNN
-F 1 "GND" H 5455 2327 50  0000 C CNN
-F 2 "" H 5450 2500 50  0001 C CNN
-F 3 "" H 5450 2500 50  0001 C CNN
-	1    5450 2500
-	1    0    0    -1
-$EndComp
-Wire Wire Line
-	7000 2600 7000 2800
 Connection ~ 7600 2700
 Wire Wire Line
 	7600 2700 8000 2700
-Wire Wire Line
-	7300 2600 7300 2700
 $Comp
 L Device:R R307
@@
 	5900 2800 5900 2700
 Connection ~ 5900 2700
-Wire Wire Line
-	5150 2300 5100 2300
-Wire Wire Line
-	5100 2300 5100 3200
 Wire Wire Line
 	6200 2800 6200 2700
@@
 Wire Wire Line
 	7000 4100 7400 4100
-$Comp
-L symbols:+VSD #PWR0118
-U 1 1 5E923782
-P 7300 2600
-F 0 "#PWR0118" H 7300 2450 50  0001 C CNN
-F 1 "+VSD" H 7315 2773 50  0000 C CNN
-F 2 "" H 7300 2600 50  0001 C CNN
-F 3 "" H 7300 2600 50  0001 C CNN
-	1    7300 2600
-	1    0    0    -1
-$EndComp
 Connection ~ 7300 2700
 Wire Wire Line
 	7300 2700 7600 2700
 Wire Wire Line
-	6500 2700 7300 2700
+	6500 2700 7000 2700
 Wire Wire Line
 	7300 2700 7300 3500
 Wire Wire Line
 	7300 3500 7400 3500
+Wire Wire Line
+	7000 2600 7000 2700
+Connection ~ 7000 2700
+Wire Wire Line
+	7000 2700 7300 2700
+Wire Wire Line
+	7000 2800 7000 2700
 $EndSCHEMATC
